Commit message: Make the wheels appear in gazebo

File: src/topnav_bot_description/urdf/four-wheeled.urdf.xacro (robot description, xacro)
@@ -1,5 +1,4 @@
 <?xml version="1.0"?>
 <robot name="four-wheeled" xmlns:xacro="http://www.ros.org/wiki/xacro">
-    <xacro:property name="pi" value="3.1415" />
     <xacro:property name="scale" value="5.0" />
     <xacro:property name="caseWidth" value="${0.2032 * scale}" />
@@ -37,4 +36,9 @@
         </visual>
         <xacro:default_inertial mass="2"/>
+        <collision>
+            <geometry>
+                <box size="${caseLength} ${caseWidth} ${caseHeight}"/>
+            </geometry>
+        </collision>
     </link>
     <xacro:macro name="wheel" params="prefix suffix origX origY origZ">
@@ -47,4 +51,11 @@
                 <material name="black"/>
             </visual>
+            <collision>
+                <origin rpy="${pi/2} 0 0" xyz="0 0 0"/>
+                <geometry>
+                    <cylinder length="${wheelWidth}" radius="${wheelDiam/2}"/>
+                </geometry>
+            </collision>
+            <xacro:default_inertial mass="0.15"/>
         </link>
         <joint name="${prefix}_${suffix}_wheel_to_base" type="continuous">
@@ -54,5 +65,4 @@
             <origin rpy="0 0 0" xyz="${origX} ${origY} ${origZ}"/>
         </joint>
-        <xacro:default_inertial mass="0.15"/>
     </xacro:macro>
     <xacro:wheel prefix="rear" suffix="left" origX="${-wheelToMiddleLength}" origY="${wheelToMiddleWidth}" origZ="0.0"/>
@@ -60,3 +70,8 @@
     <xacro:wheel prefix="front" suffix="left" origX="${wheelToMiddleLength}" origY="${wheelToMiddleWidth}" origZ="0.0"/>
     <xacro:wheel prefix="front" suffix="right" origX="${wheelToMiddleLength}" origY="${-wheelToMiddleWidth}" origZ="0.0"/>
+    <gazebo>
+        <plugin name="gazebo_ros_control" filename="libgazebo_ros_control.so">
+            <robotNamespace>/</robotNamespace>
+        </plugin>
+    </gazebo>
 </robot>
