Commit message: Rename four-wheeled to capo
    TODO fix capo.launch

File: src/topnav_bot_description/urdf/capo.urdf.xacro (robot description, xacro)
@@ -59,5 +59,5 @@
             <xacro:default_inertial mass="0.15"/>
         </link>
-        <joint name="${prefix}_${suffix}_wheel_to_base" type="continuous">
+        <joint name="${prefix}_${suffix}_wheel_joint" type="continuous">
             <axis rpy="0 0 0" xyz="0 1 0"/>
             <parent link="base_link"/>
@@ -65,4 +65,20 @@
             <origin rpy="0 0 0" xyz="${origX} ${origY} ${origZ}"/>
         </joint>
+        <transmission name="${prefix}_${suffix}_wheel_trans">
+            <type>transmission_interface/SimpleTransmission</type>
+            <actuator name="${prefix}_${suffix}_wheel_motor">
+                <mechanicalReduction>1</mechanicalReduction>
+            </actuator>
+            <joint name="${prefix}_${suffix}_wheel_joint">
+                <hardwareInterface>hardware_interface/VelocityJointInterface</hardwareInterface>
+            </joint>
+        </transmission>
+        <gazebo reference="${prefix}_${suffix}_wheel">
+            <mu1 value="200.0"/>
+            <mu2 value="100.0"/>
+            <kp value="10000000.0" />
+            <kd value="1.0" />
+            <material>Gazebo/Black</material>
+        </gazebo>
     </xacro:macro>
     <xacro:wheel prefix="rear" suffix="left" origX="${-wheelToMiddleLength}" origY="${wheelToMiddleWidth}" origZ="0.0"/>

Commit message: Change the scale to 1.0
      TODO fix the mass and the inertial characteristics of the robot

File: src/topnav_bot_description/urdf/capo.urdf.xacro (robot description, xacro)
@@ -1,5 +1,5 @@
 <?xml version="1.0"?>
 <robot name="four-wheeled" xmlns:xacro="http://www.ros.org/wiki/xacro">
-    <xacro:property name="scale" value="5.0" />
+    <xacro:property name="scale" value="1.0" />
     <xacro:property name="caseWidth" value="${0.2032 * scale}" />
     <xacro:property name="caseLength" value="${0.24765 * scale}" />

Commit message: Set inertial matrix proper for the cylinder (wheels)

File: src/topnav_bot_description/urdf/capo.urdf.xacro (robot description, xacro)
@@ -25,5 +25,7 @@
         <inertial>
             <mass value="${mass}" />
-            <inertia ixx="1.0" ixy="0.0" ixz="0.0" iyy="1.0" iyz="0.0" izz="1.0" />
+            <inertia ixx="1.0" ixy="0.0" ixz="0.0"
+                     iyy="1.0" iyz="0.0"
+                     izz="1.0" />
         </inertial>
     </xacro:macro>
@@ -42,5 +44,5 @@
         </collision>
     </link>
-    <xacro:macro name="wheel" params="prefix suffix origX origY origZ">
+    <xacro:macro name="wheel" params="prefix suffix origX origY origZ mass">
         <link name="${prefix}_${suffix}_wheel">
             <visual>
@@ -57,5 +59,12 @@
                 </geometry>
             </collision>
-            <xacro:default_inertial mass="0.15"/>
+            <inertial>
+                <xacro:property name="r" value="${wheelDiam/2}" />
+                <xacro:property name="h" value="${wheelWidth}" />
+                <mass value="${mass}" />
+                <inertia ixx="${(1/12)*mass*(3*r*r+h*h)}" ixy="0.0" ixz="0.0"
+                         iyy="${(1/12)*mass*(3*r*r+h*h)}" iyz="0.0"
+                         izz="${0.5*mass*r*r}" />
+            </inertial>
         </link>
         <joint name="${prefix}_${suffix}_wheel_joint" type="continuous">
@@ -82,8 +91,8 @@
         </gazebo>
     </xacro:macro>
-    <xacro:wheel prefix="rear" suffix="left" origX="${-wheelToMiddleLength}" origY="${wheelToMiddleWidth}" origZ="0.0"/>
-    <xacro:wheel prefix="rear" suffix="right" origX="${-wheelToMiddleLength}" origY="${-wheelToMiddleWidth}" origZ="0.0"/>
-    <xacro:wheel prefix="front" suffix="left" origX="${wheelToMiddleLength}" origY="${wheelToMiddleWidth}" origZ="0.0"/>
-    <xacro:wheel prefix="front" suffix="right" origX="${wheelToMiddleLength}" origY="${-wheelToMiddleWidth}" origZ="0.0"/>
+    <xacro:wheel prefix="rear" suffix="left" origX="${-wheelToMiddleLength}" origY="${wheelToMiddleWidth}" origZ="0.0" mass="0.15"/>
+    <xacro:wheel prefix="rear" suffix="right" origX="${-wheelToMiddleLength}" origY="${-wheelToMiddleWidth}" origZ="0.0" mass="0.15"/>
+    <xacro:wheel prefix="front" suffix="left" origX="${wheelToMiddleLength}" origY="${wheelToMiddleWidth}" origZ="0.0" mass="0.15"/>
+    <xacro:wheel prefix="front" suffix="right" origX="${wheelToMiddleLength}" origY="${-wheelToMiddleWidth}" origZ="0.0" mass="0.15"/>
     <gazebo>
         <plugin name="gazebo_ros_control" filename="libgazebo_ros_control.so">
