Commit message: Add the head

File: topnav_bot_description/urdf/capo.urdf.xacro (robot description, xacro)
@@ -10,4 +10,7 @@
     <xacro:property name="wheelToMiddleWidth" value="${(caseWidth + wheelWidth)/2 + wheelCaseGap}"/>
     <xacro:property name="wheelToMiddleLength" value="${caseLength/2 - 0.03 * scale}"/>
+    <xacro:property name="headDiam" value="${0.1 * scale}" />
+    <xacro:property name="headHeight" value="${0.08 * scale}" />
+    <xacro:property name="headWeight" value="${0.2 * scale}" />
     <material name="gray">
         <color rgba="0.5 0.5 0.5 1"/>
@@ -44,4 +47,55 @@
         </collision>
     </link>
+    <!-- head -->
+    <link name="head">
+        <visual>
+            <origin rpy="0 0 0" xyz="0 0 0"/>
+            <geometry>
+                <cylinder length="${headHeight}" radius="${headDiam/2}"/>
+            </geometry>
+            <material name="gray"/>
+        </visual>
+        <collision>
+            <origin rpy="0 0 0" xyz="0 0 0"/>
+            <geometry>
+                <cylinder length="${headHeight}" radius="${headDiam/2}"/>
+            </geometry>
+        </collision>
+        <inertial>
+            <xacro:property name="r" value="${headDiam/2}" />
+            <xacro:property name="h" value="${headHeight}" />
+            <xacro:property name="mass" value="${headWeight}" />
+            <mass value="${mass}" />
+            <inertia ixx="${(1/12)*mass*(3*r*r+h*h)}" ixy="0.0" ixz="0.0"
+                     iyy="${(1/12)*mass*(3*r*r+h*h)}" iyz="0.0"
+                     izz="${0.5*mass*r*r}" />
+        </inertial>
+    </link>
+    <joint name="head_swivel" type="continuous">
+        <parent link="base_link"/>
+        <child link="head"/>
+        <axis xyz="0 0 1"/>
+        <origin xyz="0 0 ${caseHeight / 2 + headHeight / 2}"/>
+        <limit effort="30" velocity="1.0"/>
+        <dynamics damping="0.0" friction="0.0"/>
+    </joint>
+    <!-- gazebo - head -->
+    <transmission name="head_swivel_trans">
+        <type>transmission_interface/SimpleTransmission</type>
+        <actuator name="$head_swivel_motor">
+            <mechanicalReduction>1</mechanicalReduction>
+        </actuator>
+        <joint name="head_swivel">
+            <hardwareInterface>hardware_interface/PositionJointInterface</hardwareInterface>
+        </joint>
+    </transmission>
+    <gazebo reference="head">
+        <mu1 value="200.0"/>
+        <mu2 value="100.0"/>
+        <kp value="10000000.0" />
+        <kd value="1.0" />
+        <material>Gazebo/Gray</material>
+    </gazebo>
+    <!-- /head -->
     <xacro:macro name="wheel" params="prefix suffix origX origY origZ mass">
         <link name="${prefix}_${suffix}_wheel">

Commit message: Scale the weights, change the inertial of the chassis, move the head to the front

File: topnav_bot_description/urdf/capo.urdf.xacro (robot description, xacro)
@@ -5,4 +5,5 @@
     <xacro:property name="caseLength" value="${0.24765 * scale}" />
     <xacro:property name="caseHeight" value="${0.1016 * scale}" />
+    <xacro:property name="caseWeight" value="${3 * scale}"/>
     <xacro:property name="wheelDiam" value="${0.12065 * scale}" />
     <xacro:property name="wheelWidth" value="${0.05 * scale}"/>
@@ -10,6 +11,7 @@
     <xacro:property name="wheelToMiddleWidth" value="${(caseWidth + wheelWidth)/2 + wheelCaseGap}"/>
     <xacro:property name="wheelToMiddleLength" value="${caseLength/2 - 0.03 * scale}"/>
+    <xacro:property name="wheelWeight" value="${0.15 * scale}" />
     <xacro:property name="headDiam" value="${0.1 * scale}" />
-    <xacro:property name="headHeight" value="${0.08 * scale}" />
+    <xacro:property name="headHeight" value="${0.04 * scale}" />
     <xacro:property name="headWeight" value="${0.2 * scale}" />
     <material name="gray">
@@ -40,5 +42,14 @@
             <material name="gray"/>
         </visual>
-        <xacro:default_inertial mass="2"/>
+        <inertial>
+            <xacro:property name="w" value="${caseWidth}" />
+            <xacro:property name="h" value="${caseHeight}" />
+            <xacro:property name="d" value="${caseLength}" />
+            <xacro:property name="m" value="${caseWeight}" />
+            <mass value="${m}" />
+            <inertia ixx="${(1/12)*m*(h*h+d*d)}" ixy="0.0" ixz="0.0"
+                     iyy="${(1/12)*m*(w*w+h*h)}" iyz="0.0"
+                     izz="${(1/12)*m*(w*w+d*d)}" />
+        </inertial>
         <collision>
             <geometry>
@@ -66,5 +77,5 @@
             <xacro:property name="h" value="${headHeight}" />
             <xacro:property name="mass" value="${headWeight}" />
-            <mass value="${mass}" />
+            <mass value="${mass}"/>
             <inertia ixx="${(1/12)*mass*(3*r*r+h*h)}" ixy="0.0" ixz="0.0"
                      iyy="${(1/12)*mass*(3*r*r+h*h)}" iyz="0.0"
@@ -76,5 +87,5 @@
         <child link="head"/>
         <axis xyz="0 0 1"/>
-        <origin xyz="0 0 ${caseHeight / 2 + headHeight / 2}"/>
+        <origin xyz="${caseLength/2 - headDiam/2} 0 ${caseHeight / 2 + headHeight / 2}"/>
         <limit effort="30" velocity="1.0"/>
         <dynamics damping="0.0" friction="0.0"/>
@@ -145,8 +156,8 @@
         </gazebo>
     </xacro:macro>
-    <xacro:wheel prefix="rear" suffix="left" origX="${-wheelToMiddleLength}" origY="${wheelToMiddleWidth}" origZ="0.0" mass="0.15"/>
-    <xacro:wheel prefix="rear" suffix="right" origX="${-wheelToMiddleLength}" origY="${-wheelToMiddleWidth}" origZ="0.0" mass="0.15"/>
-    <xacro:wheel prefix="front" suffix="left" origX="${wheelToMiddleLength}" origY="${wheelToMiddleWidth}" origZ="0.0" mass="0.15"/>
-    <xacro:wheel prefix="front" suffix="right" origX="${wheelToMiddleLength}" origY="${-wheelToMiddleWidth}" origZ="0.0" mass="0.15"/>
+    <xacro:wheel prefix="rear" suffix="left" origX="${-wheelToMiddleLength}" origY="${wheelToMiddleWidth}" origZ="0.0" mass="${wheelWeight}"/>
+    <xacro:wheel prefix="rear" suffix="right" origX="${-wheelToMiddleLength}" origY="${-wheelToMiddleWidth}" origZ="0.0" mass="${wheelWeight}"/>
+    <xacro:wheel prefix="front" suffix="left" origX="${wheelToMiddleLength}" origY="${wheelToMiddleWidth}" origZ="0.0" mass="${wheelWeight}"/>
+    <xacro:wheel prefix="front" suffix="right" origX="${wheelToMiddleLength}" origY="${-wheelToMiddleWidth}" origZ="0.0" mass="${wheelWeight}"/>
     <gazebo>
         <plugin name="gazebo_ros_control" filename="libgazebo_ros_control.so">

Commit message: Temporarily decrease the inertia of the head
      Decrease the stiffness coefficient
      Shorten the mass parameter name used in wheels' inertia

File: topnav_bot_description/urdf/capo.urdf.xacro (robot description, xacro)
@@ -76,5 +76,6 @@
             <xacro:property name="r" value="${headDiam/2}" />
             <xacro:property name="h" value="${headHeight}" />
-            <xacro:property name="mass" value="${headWeight}" />
+            <!-- TODO solve the problem of the head inertia-->
+            <xacro:property name="mass" value="${headWeight * 0.01}" />
             <mass value="${mass}"/>
             <inertia ixx="${(1/12)*mass*(3*r*r+h*h)}" ixy="0.0" ixz="0.0"
@@ -104,5 +105,5 @@
         <mu1 value="200.0"/>
         <mu2 value="100.0"/>
-        <kp value="10000000.0" />
+        <kp value="1000000.0" />
         <kd value="1.0" />
         <material>Gazebo/Gray</material>
@@ -127,8 +128,9 @@
                 <xacro:property name="r" value="${wheelDiam/2}" />
                 <xacro:property name="h" value="${wheelWidth}" />
-                <mass value="${mass}" />
-                <inertia ixx="${(1/12)*mass*(3*r*r+h*h)}" ixy="0.0" ixz="0.0"
-                         iyy="${(1/12)*mass*(3*r*r+h*h)}" iyz="0.0"
-                         izz="${0.5*mass*r*r}" />
+                <xacro:property name="m" value="${mass}" />
+                <mass value="${m}" />
+                <inertia ixx="${(1/12)*m*(3*r*r+h*h)}" ixy="0.0" ixz="0.0"
+                         iyy="${0.5*m*r*r}" iyz="0.0"
+                         izz="${(1/12)*m*(3*r*r+h*h)}" />
             </inertial>
         </link>

Commit message: Increase the weight of the body, tweak the friction coefficients

File: topnav_bot_description/urdf/capo.urdf.xacro (robot description, xacro)
@@ -5,5 +5,5 @@
     <xacro:property name="caseLength" value="${0.24765 * scale}" />
     <xacro:property name="caseHeight" value="${0.1016 * scale}" />
-    <xacro:property name="caseWeight" value="${3 * scale}"/>
+    <xacro:property name="caseWeight" value="${4 * scale}"/>
     <xacro:property name="wheelDiam" value="${0.12065 * scale}" />
     <xacro:property name="wheelWidth" value="${0.05 * scale}"/>
@@ -151,8 +151,9 @@
         </transmission>
         <gazebo reference="${prefix}_${suffix}_wheel">
-            <mu1 value="200.0"/>
-            <mu2 value="100.0"/>
-            <kp value="10000000.0" />
+            <mu value="4.0"/>
+            <mu2 value="1.0"/>
+            <kp value="1000000.0" />
             <kd value="1.0" />
+            <!--<fdir1>0 0 1</fdir1>-->
             <material>Gazebo/Black</material>
         </gazebo>
