Commit message: Place camera right behind the lidar, enable defining the initial position of the robot

File: topnav_bot_description/urdf/capo/head/capo.head.xacro (robot description, xacro)
@@ -31,5 +31,5 @@
         <child link="head"/>
         <axis xyz="0 0 1"/>
-        <origin xyz="0 0 ${caseHeight / 2 + headHeight / 2}"/>
+        <origin xyz="${caseLength / 2 - (hokuyoSide + headDiam / 2)} 0 ${caseHeight / 2 + headHeight / 2}"/>
         <limit effort="30"
                velocity="1.0"
