Commit message: Add the battery, tweak the masses and the inertial values

File: topnav_bot_description/urdf/capo/head/camera.xacro (robot description, xacro)
@@ -24,5 +24,7 @@
             <mass value="1e-5"/>
             <origin xyz="0 0 0" rpy="0 0 0"/>
-            <inertia ixx="1e-6" ixy="0" ixz="0" iyy="1e-6" iyz="0" izz="1e-6"/>
+            <inertia ixx="1e-6" ixy="0.0" ixz="0.0"
+                     iyy="1e-6" iyz="0.0"
+                     izz="1e-6" />
         </inertial>
     </link>

File: topnav_bot_description/urdf/capo2/capo2.urdf.xacro (robot description, xacro)
@@ -7,5 +7,11 @@
     <xacro:property name="caseLength" value="${0.18 * scale}" />
     <xacro:property name="caseHeight" value="${0.12 * scale}" />
-    <xacro:property name="caseWeight" value="${4 * scale}"/>
+    <xacro:property name="caseWeight" value="${1.0 * scale}"/>
+    <xacro:property name="batteryWidth" value="${0.13 * scale}" />
+    <xacro:property name="batteryLength" value="${0.04 * scale}" />
+    <xacro:property name="batteryHeight" value="${0.05 * scale}" />
+    <xacro:property name="batteryWeight" value="${0.5 * scale}"/>
+    <xacro:property name="batteryOffset" value="${-0.065 * scale}" />
+    <xacro:property name="batteryHeightOffset" value="${-0.03 * scale}" />
     <xacro:property name="wheelDiam" value="${0.09 * scale}" />
     <xacro:property name="wheelWidth" value="${0.01 * scale}"/>
@@ -26,5 +32,5 @@
     <xacro:property name="hokuyoHeightOffset" value="${0.03 * scale}" />
     <xacro:property name="casterWheelRadius" value="${0.01 * scale}"/>
-    <xacro:property name="casterWheelWeight" value="${1.0 * scale}"/>
+    <xacro:property name="casterWheelWeight" value="${0.5 * scale}"/>
     <xacro:property name="laserSamplesCount" value="61"/>
     <xacro:property name="laserMinAngle" value="${-2*pi/3}"/>
@@ -68,4 +74,41 @@
         </collision>
     </link>
+    <gazebo reference="base_link">
+        <material>Gazebo/Wood</material>
+    </gazebo>
+    <!--battery -->
+    <link name ="battery">
+        <visual>
+            <geometry>
+                <box size="${batteryLength} ${batteryWidth} ${batteryHeight}"/>
+            </geometry>
+            <material name="gray"/>
+        </visual>
+        <inertial>
+            <xacro:property name="w" value="${batteryWidth}" />
+            <xacro:property name="h" value="${batteryHeight}" />
+            <xacro:property name="d" value="${batteryLength}" />
+            <xacro:property name="m" value="${batteryWeight}" />
+            <mass value="${m}" />
+            <inertia ixx="${(1/12)*m*(h*h+d*d)}" ixy="0.0" ixz="0.0"
+                     iyy="${(1/12)*m*(w*w+h*h)}" iyz="0.0"
+                     izz="${(1/12)*m*(w*w+d*d)}" />
+        </inertial>
+        <collision>
+            <geometry>
+                <box size="${batteryLength} ${batteryWidth} ${batteryHeight}"/>
+            </geometry>
+        </collision>
+    </link>
+    <joint name="base_battery_joint" type="fixed">
+        <axis rpy="0 0 0" xyz="0 1 0"/>
+        <parent link="base_link"/>
+        <child link="battery"/>
+        <origin rpy="0 0 0" xyz="${batteryOffset} 0.0 ${batteryHeightOffset}"/>
+    </joint>
+    <gazebo reference="battery">
+        <material>Gazebo/Blue</material>
+    </gazebo>
+    <!-- battery -->
     <xacro:include filename="../capo/head/capo.head.xacro" />
     <transmission name="head_swivel_trans">
@@ -133,5 +176,5 @@
             <mu1 value="40.0"/>
             <mu2 value="20.0"/>
-            <kp value="1000000.0" />
+            <kp value="10000000.0" />
             <kd value="1.0" />
             <!--<fdir1>0 0 1</fdir1>-->
@@ -141,6 +184,6 @@
         </gazebo>
     </xacro:macro>
-    <xacro:wheel prefix="rear" suffix="left" origX="${-wheelToMiddleLength}" origY="${wheelToMiddleWidth}" origZ="0.0" mass="${wheelWeight}" diam="0.01" width="0.01"/>
-    <xacro:wheel prefix="rear" suffix="right" origX="${-wheelToMiddleLength}" origY="${-wheelToMiddleWidth}" origZ="0.0" mass="${wheelWeight}" diam="0.01" width="0.01"/>
+    <xacro:wheel prefix="rear" suffix="left" origX="${-wheelToMiddleLength}" origY="${wheelToMiddleWidth}" origZ="0.0" mass="${wheelWeight * 0.0001}" diam="0.01" width="0.01"/>
+    <xacro:wheel prefix="rear" suffix="right" origX="${-wheelToMiddleLength}" origY="${-wheelToMiddleWidth}" origZ="0.0" mass="${wheelWeight * 0.0001}" diam="0.01" width="0.01"/>
     <xacro:wheel prefix="front" suffix="left" origX="${wheelToMiddleLength}" origY="${wheelToMiddleWidth}" origZ="-0.025" mass="${wheelWeight}" diam="${wheelDiam}" width="${wheelWidth}"/>
     <xacro:wheel prefix="front" suffix="right" origX="${wheelToMiddleLength}" origY="${-wheelToMiddleWidth}" origZ="-0.025" mass="${wheelWeight}" diam="${wheelDiam}" width="${wheelWidth}"/>
@@ -184,6 +227,7 @@
         </joint>
     </xacro:macro>
-    <xacro:caster_wheel prefix="left" origX="-0.08" origY="0.04" origZ="${scale * -0.06}"/>
-    <xacro:caster_wheel prefix="right" origX="-0.08" origY="-0.04" origZ="${scale * -0.06}"/>
+    <!--<xacro:caster_wheel prefix="left" origX="-0.08" origY="0.04" origZ="${scale * -0.06}"/>-->
+    <!--<xacro:caster_wheel prefix="right" origX="-0.08" origY="-0.04" origZ="${scale * -0.06}"/>-->
+    <xacro:caster_wheel prefix="center" origX="-0.08" origY="0.0" origZ="${scale * -0.06}"/>
     <gazebo>
         <plugin name="gazebo_ros_control" filename="libgazebo_ros_control.so">
