Commit message: Move parts of the robot model to the separate files

File: topnav_bot_description/urdf/capo/capo.urdf.xacro (robot description, xacro)
@@ -58,39 +58,5 @@
         </collision>
     </link>
-    <!-- head -->
-    <link name="head">
-        <visual>
-            <origin rpy="0 0 0" xyz="0 0 0"/>
-            <geometry>
-                <cylinder length="${headHeight}" radius="${headDiam/2}"/>
-            </geometry>
-            <material name="gray"/>
-        </visual>
-        <collision>
-            <origin rpy="0 0 0" xyz="0 0 0"/>
-            <geometry>
-                <cylinder length="${headHeight}" radius="${headDiam/2}"/>
-            </geometry>
-        </collision>
-        <inertial>
-            <xacro:property name="r" value="${headDiam/2}" />
-            <xacro:property name="h" value="${headHeight}" />
-            <!-- TODO solve the problem of the head inertia-->
-            <xacro:property name="mass" value="${headWeight * 0.01}" />
-            <mass value="${mass}"/>
-            <inertia ixx="${(1/12)*mass*(3*r*r+h*h)}" ixy="0.0" ixz="0.0"
-                     iyy="${(1/12)*mass*(3*r*r+h*h)}" iyz="0.0"
-                     izz="${0.5*mass*r*r}" />
-        </inertial>
-    </link>
-    <joint name="head_swivel" type="continuous">
-        <parent link="base_link"/>
-        <child link="head"/>
-        <axis xyz="0 0 1"/>
-        <origin xyz="${caseLength/2 - headDiam/2} 0 ${caseHeight / 2 + headHeight / 2}"/>
-        <limit effort="30" velocity="1.0"/>
-        <dynamics damping="0.0" friction="0.0"/>
-    </joint>
-    <!-- gazebo - head -->
+    <xacro:include filename="head/capo.head.xacro" />
     <transmission name="head_swivel_trans">
         <type>transmission_interface/SimpleTransmission</type>

Commit message: Change camera's dimensions and position

File: topnav_bot_description/urdf/capo/capo.urdf.xacro (robot description, xacro)
@@ -15,4 +15,7 @@
     <xacro:property name="headHeight" value="${0.04 * scale}" />
     <xacro:property name="headWeight" value="${0.2 * scale}" />
+    <xacro:property name="cameraWidth" value="${0.095 * scale}" />
+    <xacro:property name="cameraHeight" value="${0.03 * scale}" />
+    <xacro:property name="cameraDepth" value="${0.03 * scale}" />
     <material name="gray">
         <color rgba="0.5 0.5 0.5 1"/>

File: topnav_bot_description/urdf/capo/head/capo.head.xacro (robot description, xacro)
@@ -1,4 +1,5 @@
 <robot xmlns:xacro="http://www.ros.org/wiki/xacro">
     <!-- head -->
+    <xacro:property name="camera_link" value="0.05" />
     <link name="head">
         <visual>
@@ -35,3 +36,4 @@
     </joint>
     <!-- gazebo - head -->
+   <xacro:include filename="camera.xacro"/>
 </robot>

Commit message: Add Hokuyo laser scanner

File: topnav_bot_description/urdf/capo/capo.urdf.xacro (robot description, xacro)
@@ -18,4 +18,6 @@
     <xacro:property name="cameraHeight" value="${0.03 * scale}" />
     <xacro:property name="cameraDepth" value="${0.03 * scale}" />
+    <xacro:property name="hokuyoSide" value="${0.05 * scale}" />
+    <xacro:property name="hokuyoHeight" value="${0.07 * scale}" />
     <material name="gray">
         <color rgba="0.5 0.5 0.5 1"/>

File: topnav_bot_description/urdf/capo/head/capo.head.xacro (robot description, xacro)
@@ -1,5 +1,5 @@
 <robot xmlns:xacro="http://www.ros.org/wiki/xacro">
     <!-- head -->
-    <xacro:property name="camera_link" value="0.05" />
+    <xacro:property name="camera_link" value="0.05"/>
     <link name="head">
         <visual>
@@ -36,4 +36,5 @@
     </joint>
     <!-- gazebo - head -->
-   <xacro:include filename="camera.xacro"/>
+    <xacro:include filename="camera.xacro"/>
+    <xacro:include filename="hokuyo.xacro"/>
 </robot>

Commit message: Feature/sensors (#1)
* Add the head

* Scale the weights, change the inertial of the chassis, move the head to the front

* Add publisher and subscriber from the tutorial

* Send and empty message, move topic name to the header file

* Simplify imports

* Enable the creation of ResetWorld service

* Send reset model signal

* Temporarily decrease the inertia of the head

      Decrease the stiffness coefficient
      Shorten the mass parameter name used in wheels' inertia

* Increase the weight of the body, tweak the friction coefficients

* Move parts of the robot model to the separate files

* Change camera's dimensions and position

* Capture images from the camera

* Add Hokuyo laser scanner

* Fix missing links of the included files, show the laser beam

* Change laser scan range
      Minimum 20cm
      Maximum 5m

File: topnav_bot_description/urdf/capo/capo.urdf.xacro (robot description, xacro)
@@ -5,4 +5,5 @@
     <xacro:property name="caseLength" value="${0.24765 * scale}" />
     <xacro:property name="caseHeight" value="${0.1016 * scale}" />
+    <xacro:property name="caseWeight" value="${4 * scale}"/>
     <xacro:property name="wheelDiam" value="${0.12065 * scale}" />
     <xacro:property name="wheelWidth" value="${0.05 * scale}"/>
@@ -10,4 +11,13 @@
     <xacro:property name="wheelToMiddleWidth" value="${(caseWidth + wheelWidth)/2 + wheelCaseGap}"/>
     <xacro:property name="wheelToMiddleLength" value="${caseLength/2 - 0.03 * scale}"/>
+    <xacro:property name="wheelWeight" value="${0.15 * scale}" />
+    <xacro:property name="headDiam" value="${0.1 * scale}" />
+    <xacro:property name="headHeight" value="${0.04 * scale}" />
+    <xacro:property name="headWeight" value="${0.2 * scale}" />
+    <xacro:property name="cameraWidth" value="${0.095 * scale}" />
+    <xacro:property name="cameraHeight" value="${0.03 * scale}" />
+    <xacro:property name="cameraDepth" value="${0.03 * scale}" />
+    <xacro:property name="hokuyoSide" value="${0.05 * scale}" />
+    <xacro:property name="hokuyoHeight" value="${0.07 * scale}" />
     <material name="gray">
         <color rgba="0.5 0.5 0.5 1"/>
@@ -37,5 +47,14 @@
             <material name="gray"/>
         </visual>
-        <xacro:default_inertial mass="2"/>
+        <inertial>
+            <xacro:property name="w" value="${caseWidth}" />
+            <xacro:property name="h" value="${caseHeight}" />
+            <xacro:property name="d" value="${caseLength}" />
+            <xacro:property name="m" value="${caseWeight}" />
+            <mass value="${m}" />
+            <inertia ixx="${(1/12)*m*(h*h+d*d)}" ixy="0.0" ixz="0.0"
+                     iyy="${(1/12)*m*(w*w+h*h)}" iyz="0.0"
+                     izz="${(1/12)*m*(w*w+d*d)}" />
+        </inertial>
         <collision>
             <geometry>
@@ -44,4 +63,22 @@
         </collision>
     </link>
+    <xacro:include filename="head/capo.head.xacro" />
+    <transmission name="head_swivel_trans">
+        <type>transmission_interface/SimpleTransmission</type>
+        <actuator name="$head_swivel_motor">
+            <mechanicalReduction>1</mechanicalReduction>
+        </actuator>
+        <joint name="head_swivel">
+            <hardwareInterface>hardware_interface/PositionJointInterface</hardwareInterface>
+        </joint>
+    </transmission>
+    <gazebo reference="head">
+        <mu1 value="200.0"/>
+        <mu2 value="100.0"/>
+        <kp value="1000000.0" />
+        <kd value="1.0" />
+        <material>Gazebo/Gray</material>
+    </gazebo>
+    <!-- /head -->
     <xacro:macro name="wheel" params="prefix suffix origX origY origZ mass">
         <link name="${prefix}_${suffix}_wheel">
@@ -62,8 +99,9 @@
                 <xacro:property name="r" value="${wheelDiam/2}" />
                 <xacro:property name="h" value="${wheelWidth}" />
-                <mass value="${mass}" />
-                <inertia ixx="${(1/12)*mass*(3*r*r+h*h)}" ixy="0.0" ixz="0.0"
-                         iyy="${(1/12)*mass*(3*r*r+h*h)}" iyz="0.0"
-                         izz="${0.5*mass*r*r}" />
+                <xacro:property name="m" value="${mass}" />
+                <mass value="${m}" />
+                <inertia ixx="${(1/12)*m*(3*r*r+h*h)}" ixy="0.0" ixz="0.0"
+                         iyy="${0.5*m*r*r}" iyz="0.0"
+                         izz="${(1/12)*m*(3*r*r+h*h)}" />
             </inertial>
         </link>
@@ -84,15 +122,16 @@
         </transmission>
         <gazebo reference="${prefix}_${suffix}_wheel">
-            <mu1 value="200.0"/>
-            <mu2 value="100.0"/>
-            <kp value="10000000.0" />
+            <mu value="4.0"/>
+            <mu2 value="1.0"/>
+            <kp value="1000000.0" />
             <kd value="1.0" />
+            <!--<fdir1>0 0 1</fdir1>-->
             <material>Gazebo/Black</material>
         </gazebo>
     </xacro:macro>
-    <xacro:wheel prefix="rear" suffix="left" origX="${-wheelToMiddleLength}" origY="${wheelToMiddleWidth}" origZ="0.0" mass="0.15"/>
-    <xacro:wheel prefix="rear" suffix="right" origX="${-wheelToMiddleLength}" origY="${-wheelToMiddleWidth}" origZ="0.0" mass="0.15"/>
-    <xacro:wheel prefix="front" suffix="left" origX="${wheelToMiddleLength}" origY="${wheelToMiddleWidth}" origZ="0.0" mass="0.15"/>
-    <xacro:wheel prefix="front" suffix="right" origX="${wheelToMiddleLength}" origY="${-wheelToMiddleWidth}" origZ="0.0" mass="0.15"/>
+    <xacro:wheel prefix="rear" suffix="left" origX="${-wheelToMiddleLength}" origY="${wheelToMiddleWidth}" origZ="0.0" mass="${wheelWeight}"/>
+    <xacro:wheel prefix="rear" suffix="right" origX="${-wheelToMiddleLength}" origY="${-wheelToMiddleWidth}" origZ="0.0" mass="${wheelWeight}"/>
+    <xacro:wheel prefix="front" suffix="left" origX="${wheelToMiddleLength}" origY="${wheelToMiddleWidth}" origZ="0.0" mass="${wheelWeight}"/>
+    <xacro:wheel prefix="front" suffix="right" origX="${wheelToMiddleLength}" origY="${-wheelToMiddleWidth}" origZ="0.0" mass="${wheelWeight}"/>
     <gazebo>
         <plugin name="gazebo_ros_control" filename="libgazebo_ros_control.so">

Commit message: Move laser parameters to the main file
      * Move some publisher and subscriber stuff for the line follower

File: topnav_bot_description/urdf/capo/capo.urdf.xacro (robot description, xacro)
@@ -20,4 +20,7 @@
     <xacro:property name="hokuyoSide" value="${0.05 * scale}" />
     <xacro:property name="hokuyoHeight" value="${0.07 * scale}" />
+    <xacro:property name="laserSamplesCount" value="180"/>
+    <xacro:property name="laserMinAngle" value="${-pi/2}"/>
+    <xacro:property name="laserMaxAngle" value="${pi/2}"/>
     <material name="gray">
         <color rgba="0.5 0.5 0.5 1"/>

Commit message: Print accumulator, fix wrong angle and range parameters' order

File: topnav_bot_description/urdf/capo/capo.urdf.xacro (robot description, xacro)
@@ -20,5 +20,5 @@
     <xacro:property name="hokuyoSide" value="${0.05 * scale}" />
     <xacro:property name="hokuyoHeight" value="${0.07 * scale}" />
-    <xacro:property name="laserSamplesCount" value="180"/>
+    <xacro:property name="laserSamplesCount" value="45"/>
     <xacro:property name="laserMinAngle" value="${-pi/2}"/>
     <xacro:property name="laserMaxAngle" value="${pi/2}"/>

Commit message: Increase laser scan range to 240 degrees
      * Change samples count to 61 (60 gaps, 4 degrees each)

File: topnav_bot_description/urdf/capo/capo.urdf.xacro (robot description, xacro)
@@ -20,7 +20,7 @@
     <xacro:property name="hokuyoSide" value="${0.05 * scale}" />
     <xacro:property name="hokuyoHeight" value="${0.07 * scale}" />
-    <xacro:property name="laserSamplesCount" value="45"/>
-    <xacro:property name="laserMinAngle" value="${-pi/2}"/>
-    <xacro:property name="laserMaxAngle" value="${pi/2}"/>
+    <xacro:property name="laserSamplesCount" value="61"/>
+    <xacro:property name="laserMinAngle" value="${-2*pi/3}"/>
+    <xacro:property name="laserMaxAngle" value="${2*pi/3}"/>
     <material name="gray">
         <color rgba="0.5 0.5 0.5 1"/>

Commit message: Move head to the center, attach the lidar directly to the case

File: topnav_bot_description/urdf/capo/capo.urdf.xacro (robot description, xacro)
@@ -13,5 +13,5 @@
     <xacro:property name="wheelWeight" value="${0.15 * scale}" />
     <xacro:property name="headDiam" value="${0.1 * scale}" />
-    <xacro:property name="headHeight" value="${0.04 * scale}" />
+    <xacro:property name="headHeight" value="${0.08 * scale}" />
     <xacro:property name="headWeight" value="${0.2 * scale}" />
     <xacro:property name="cameraWidth" value="${0.095 * scale}" />

File: topnav_bot_description/urdf/capo/head/capo.head.xacro (robot description, xacro)
@@ -27,10 +27,13 @@
         </inertial>
     </link>
-    <joint name="head_swivel" type="continuous">
+    <joint name="head_swivel" type="revolute">
         <parent link="base_link"/>
         <child link="head"/>
         <axis xyz="0 0 1"/>
-        <origin xyz="${caseLength/2 - headDiam/2} 0 ${caseHeight / 2 + headHeight / 2}"/>
-        <limit effort="30" velocity="1.0"/>
+        <origin xyz="0 0 ${caseHeight / 2 + headHeight / 2}"/>
+        <limit effort="30"
+               velocity="1.0"
+               lower="-2.0944"
+               upper="2.0944"/>
         <dynamics damping="0.0" friction="0.0"/>
     </joint>

File: topnav_bot_description/urdf/capo/head/hokuyo.xacro (robot description, xacro)
@@ -2,6 +2,6 @@
     <joint name="hokuyo_joint" type="fixed">
         <axis xyz="0 1 0"/>
-        <origin xyz="0 0 ${headHeight/2 + hokuyoHeight/2}" rpy="0 0 0"/>
-        <parent link="head"/>
+        <origin xyz="${caseLength/2 - hokuyoSide/2} 0 ${caseHeight/2 + hokuyoHeight/2}" rpy="0 0 0"/>
+        <parent link="base_link"/>
         <child link="hokuyo_link"/>
     </joint>

Commit message: Specify the clusters count and the angle range
      * Samples count: 62
      * Angle range: ca. 238 deg

File: topnav_bot_description/urdf/capo/capo.urdf.xacro (robot description, xacro)
@@ -21,7 +21,7 @@
     <xacro:property name="hokuyoSide" value="${0.05 * scale}" />
     <xacro:property name="hokuyoHeight" value="${0.07 * scale}" />
-    <xacro:property name="laserSamplesCount" value="61"/>
-    <xacro:property name="laserMinAngle" value="${-2*pi/3}"/>
-    <xacro:property name="laserMaxAngle" value="${2*pi/3}"/>
+    <xacro:property name="laserSamplesCount" value="62"/>
+    <xacro:property name="laserMinAngle" value="-2.08"/>
+    <xacro:property name="laserMaxAngle" value="2.08"/>
     <xacro:macro name="default_inertial" params="mass">
         <inertial>

Commit message: Decrease the camera's resolution, update the robot's model

File: topnav_bot_description/urdf/capo/capo.urdf.xacro (robot description, xacro)
@@ -16,4 +16,5 @@
     <xacro:property name="headHeight" value="${0.08 * scale}" />
     <xacro:property name="headWeight" value="${0.2 * scale}" />
+    <xacro:property name="headOffset" value="${0.0 * scale}" />
     <xacro:property name="cameraWidth" value="${0.095 * scale}" />
     <xacro:property name="cameraHeight" value="${0.03 * scale}" />
@@ -21,4 +22,5 @@
     <xacro:property name="hokuyoSide" value="${0.05 * scale}" />
     <xacro:property name="hokuyoHeight" value="${0.07 * scale}" />
+    <xacro:property name="hokuyoOffset" value="${0.0 * scale}" />
     <xacro:property name="laserSamplesCount" value="62"/>
     <xacro:property name="laserMinAngle" value="-2.08"/>

File: topnav_bot_description/urdf/capo/head/capo.head.xacro (robot description, xacro)
@@ -31,5 +31,5 @@
         <child link="head"/>
         <axis xyz="0 0 1"/>
-        <origin xyz="${caseLength / 2 - (hokuyoSide + headDiam / 2)} 0 ${caseHeight / 2 + headHeight / 2}"/>
+        <origin xyz="${caseLength / 2 - (hokuyoSide + headDiam / 2 + headOffset)} 0 ${caseHeight / 2 + headHeight / 2}"/>
         <limit effort="30"
                velocity="1.0"

File: topnav_bot_description/urdf/capo/head/hokuyo.xacro (robot description, xacro)
@@ -2,5 +2,5 @@
     <joint name="hokuyo_joint" type="fixed">
         <axis xyz="0 1 0"/>
-        <origin xyz="${caseLength/2 - hokuyoSide/2} 0 ${caseHeight/2 + hokuyoHeight/2}" rpy="0 0 0"/>
+        <origin xyz="${caseLength/2 - (hokuyoSide/2 + hokuyoOffset)} 0 ${caseHeight/2 + hokuyoHeight/2}" rpy="0 0 0"/>
         <parent link="base_link"/>
         <child link="hokuyo_link"/>

File: topnav_bot_description/urdf/capo2/capo2.urdf.xacro (robot description, xacro)
@@ -3,10 +3,10 @@
     <xacro:include filename="$(find topnav_bot_description)/urdf/materials.xacro" />
     <xacro:property name="scale" value="1.0" />
-    <xacro:property name="caseWidth" value="${0.1 * scale}" />
+    <xacro:property name="caseWidth" value="${0.135 * scale}" />
     <xacro:property name="caseLength" value="${0.18 * scale}" />
     <xacro:property name="caseHeight" value="${0.12 * scale}" />
     <xacro:property name="caseWeight" value="${4 * scale}"/>
-    <xacro:property name="wheelDiam" value="${0.1 * scale}" />
-    <xacro:property name="wheelWidth" value="${0.02 * scale}"/>
+    <xacro:property name="wheelDiam" value="${0.09 * scale}" />
+    <xacro:property name="wheelWidth" value="${0.01 * scale}"/>
     <xacro:property name="wheelCaseGap" value="${0.0008 * scale}"/>
     <xacro:property name="wheelToMiddleWidth" value="${(caseWidth + wheelWidth)/2 + wheelCaseGap}"/>
@@ -16,4 +16,5 @@
     <xacro:property name="headHeight" value="${0.08 * scale}" />
     <xacro:property name="headWeight" value="${0.1 * scale}" />
+    <xacro:property name="headOffset" value="${0.07 * scale}" />
     <xacro:property name="cameraWidth" value="${0.095 * scale}" />
     <xacro:property name="cameraHeight" value="${0.03 * scale}" />
@@ -21,4 +22,5 @@
     <xacro:property name="hokuyoSide" value="${0.05 * scale}" />
     <xacro:property name="hokuyoHeight" value="${0.07 * scale}" />
+    <xacro:property name="hokuyoOffset" value="${0.03 * scale}" />
     <xacro:property name="casterWheelRadius" value="${0.01 * scale}"/>
     <xacro:property name="casterWheelWeight" value="${0.1* scale}"/>
@@ -130,6 +132,6 @@
     <xacro:wheel prefix="rear" suffix="left" origX="${-wheelToMiddleLength}" origY="${wheelToMiddleWidth}" origZ="0.0" mass="${wheelWeight}" diam="0.01" width="0.01"/>
     <xacro:wheel prefix="rear" suffix="right" origX="${-wheelToMiddleLength}" origY="${-wheelToMiddleWidth}" origZ="0.0" mass="${wheelWeight}" diam="0.01" width="0.01"/>
-    <xacro:wheel prefix="front" suffix="left" origX="${wheelToMiddleLength}" origY="${wheelToMiddleWidth}" origZ="-0.02" mass="${wheelWeight}" diam="${wheelDiam}" width="${wheelWidth}"/>
-    <xacro:wheel prefix="front" suffix="right" origX="${wheelToMiddleLength}" origY="${-wheelToMiddleWidth}" origZ="-0.02" mass="${wheelWeight}" diam="${wheelDiam}" width="${wheelWidth}"/>
+    <xacro:wheel prefix="front" suffix="left" origX="${wheelToMiddleLength}" origY="${wheelToMiddleWidth}" origZ="-0.025" mass="${wheelWeight}" diam="${wheelDiam}" width="${wheelWidth}"/>
+    <xacro:wheel prefix="front" suffix="right" origX="${wheelToMiddleLength}" origY="${-wheelToMiddleWidth}" origZ="-0.025" mass="${wheelWeight}" diam="${wheelDiam}" width="${wheelWidth}"/>
     <xacro:macro name="caster_wheel" params="prefix origX origY origZ">
         <link name="${prefix}_caster_wheel">

Commit message: Lower the LIDAR's height placement, set the camera's pitch to 0
      * Move the preview dimensions to the constants

File: topnav_bot_description/urdf/capo/capo.urdf.xacro (robot description, xacro)
@@ -23,4 +23,5 @@
     <xacro:property name="hokuyoHeight" value="${0.07 * scale}" />
     <xacro:property name="hokuyoOffset" value="${0.0 * scale}" />
+    <xacro:property name="hokuyoHeightOffset" value="${0.0 * scale}" />
     <xacro:property name="laserSamplesCount" value="62"/>
     <xacro:property name="laserMinAngle" value="-2.08"/>

File: topnav_bot_description/urdf/capo/head/hokuyo.xacro (robot description, xacro)
@@ -2,5 +2,5 @@
     <joint name="hokuyo_joint" type="fixed">
         <axis xyz="0 1 0"/>
-        <origin xyz="${caseLength/2 - (hokuyoSide/2 + hokuyoOffset)} 0 ${caseHeight/2 + hokuyoHeight/2}" rpy="0 0 0"/>
+        <origin xyz="${caseLength/2 - (hokuyoSide/2 + hokuyoOffset)} 0 ${caseHeight/2 + hokuyoHeight/2 - hokuyoHeightOffset}" rpy="0 0 0"/>
         <parent link="base_link"/>
         <child link="hokuyo_link"/>

File: topnav_bot_description/urdf/capo2/capo2.urdf.xacro (robot description, xacro)
@@ -23,4 +23,5 @@
     <xacro:property name="hokuyoHeight" value="${0.07 * scale}" />
     <xacro:property name="hokuyoOffset" value="${0.03 * scale}" />
+    <xacro:property name="hokuyoHeightOffset" value="${0.03 * scale}" />
     <xacro:property name="casterWheelRadius" value="${0.01 * scale}"/>
     <xacro:property name="casterWheelWeight" value="${0.1* scale}"/>

Commit message: Allow to use real camera during the simulation
      * In order to simulate the latency
      * Set use_real_camera to true for capo.launch
      * use the webcam (e.g. Logitech c930) to capture the displayed
      * ... capo/camera_real/image_raw
      * run the opencv_videostream

File: topnav_bot_description/urdf/capo/capo.urdf.xacro (robot description, xacro)
@@ -2,4 +2,5 @@
 <robot name="capo" xmlns:xacro="http://www.ros.org/wiki/xacro">
     <xacro:include filename="$(find topnav_bot_description)/urdf/materials.xacro" />
+    <xacro:arg name="use_sim_camera" default="false" />
     <xacro:property name="scale" value="1.0" />
     <xacro:property name="caseWidth" value="${0.2032 * scale}" />
@@ -27,4 +28,10 @@
     <xacro:property name="laserMinAngle" value="-2.08"/>
     <xacro:property name="laserMaxAngle" value="2.08"/>
+    <xacro:if value="$(arg use_real_camera)">
+        <xacro:property name="cameraFileName" value="camera_sim.gazebo" />
+    </xacro:if>
+    <xacro:unless value="$(arg use_real_camera)">
+        <xacro:property name="cameraFileName" value="camera.gazebo" />
+    </xacro:unless>
     <xacro:macro name="default_inertial" params="mass">
         <inertial>

File: topnav_bot_description/urdf/capo/head/camera.xacro (robot description, xacro)
@@ -27,4 +27,4 @@
         </inertial>
     </link>
-    <xacro:include filename="camera.gazebo" />
+    <xacro:include filename="${cameraFileName}" />
 </robot>

File: topnav_bot_description/urdf/capo2/capo2.urdf.xacro (robot description, xacro)
@@ -2,4 +2,5 @@
 <robot name="capo" xmlns:xacro="http://www.ros.org/wiki/xacro">
     <xacro:include filename="$(find topnav_bot_description)/urdf/materials.xacro" />
+    <xacro:arg name="use_real_camera" default="false" />
     <xacro:property name="scale" value="1.0" />
     <xacro:property name="caseWidth" value="${0.135 * scale}" />
@@ -29,4 +30,10 @@
     <xacro:property name="laserMinAngle" value="${-2*pi/3}"/>
     <xacro:property name="laserMaxAngle" value="${2*pi/3}"/>
+    <xacro:if value="$(arg use_real_camera)">
+        <xacro:property name="cameraFileName" value="camera_real.gazebo" />
+    </xacro:if>
+    <xacro:unless value="$(arg use_real_camera)">
+        <xacro:property name="cameraFileName" value="camera.gazebo" />
+    </xacro:unless>
     <xacro:macro name="default_inertial" params="mass">
         <inertial>
