Commit message: Add the castor wheel, switch to capo2 in all of the tests

File: topnav_bot_description/urdf/capo2/capo2.urdf.xacro (robot description, xacro)
@@ -3,15 +3,15 @@
     <xacro:include filename="$(find topnav_bot_description)/urdf/materials.xacro" />
     <xacro:property name="scale" value="1.0" />
-    <xacro:property name="caseWidth" value="${0.2032 * scale}" />
-    <xacro:property name="caseLength" value="${0.24765 * scale}" />
-    <xacro:property name="caseHeight" value="${0.1016 * scale}" />
+    <xacro:property name="caseWidth" value="${0.1 * scale}" />
+    <xacro:property name="caseLength" value="${0.18 * scale}" />
+    <xacro:property name="caseHeight" value="${0.12 * scale}" />
     <xacro:property name="caseWeight" value="${4 * scale}"/>
-    <xacro:property name="wheelDiam" value="${0.12065 * scale}" />
-    <xacro:property name="wheelWidth" value="${0.05 * scale}"/>
+    <xacro:property name="wheelDiam" value="${0.1 * scale}" />
+    <xacro:property name="wheelWidth" value="${0.005 * scale}"/>
     <xacro:property name="wheelCaseGap" value="${0.0008 * scale}"/>
     <xacro:property name="wheelToMiddleWidth" value="${(caseWidth + wheelWidth)/2 + wheelCaseGap}"/>
-    <xacro:property name="wheelToMiddleLength" value="${caseLength/2 - 0.03 * scale}"/>
+    <xacro:property name="wheelToMiddleLength" value="${caseLength/2 - 0.06 * scale}"/>
     <xacro:property name="wheelWeight" value="${0.15 * scale}" />
-    <xacro:property name="headDiam" value="${0.1 * scale}" />
+    <xacro:property name="headDiam" value="${0.05 * scale}" />
     <xacro:property name="headHeight" value="${0.08 * scale}" />
     <xacro:property name="headWeight" value="${0.2 * scale}" />
@@ -21,4 +21,6 @@
     <xacro:property name="hokuyoSide" value="${0.05 * scale}" />
     <xacro:property name="hokuyoHeight" value="${0.07 * scale}" />
+    <xacro:property name="casterWheelRadius" value="${0.01 * scale}"/>
+    <xacro:property name="casterWheelWeight" value="${0.005 * scale}"/>
     <xacro:property name="laserSamplesCount" value="61"/>
     <xacro:property name="laserMinAngle" value="${-2*pi/3}"/>
@@ -75,10 +77,10 @@
     </gazebo>
     <!-- /head -->
-    <xacro:macro name="wheel" params="prefix suffix origX origY origZ mass">
+    <xacro:macro name="wheel" params="prefix suffix origX origY origZ mass diam width">
         <link name="${prefix}_${suffix}_wheel">
             <visual>
                 <origin rpy="${pi/2} 0 0" xyz="0 0 0"/>
                 <geometry>
-                    <cylinder length="${wheelWidth}" radius="${wheelDiam/2}"/>
+                    <cylinder length="${width}" radius="${diam/2}"/>
                 </geometry>
                 <material name="black"/>
@@ -87,10 +89,10 @@
                 <origin rpy="${pi/2} 0 0" xyz="0 0 0"/>
                 <geometry>
-                    <cylinder length="${wheelWidth}" radius="${wheelDiam/2}"/>
+                    <cylinder length="${width}" radius="${diam/2}"/>
                 </geometry>
             </collision>
             <inertial>
-                <xacro:property name="r" value="${wheelDiam/2}" />
-                <xacro:property name="h" value="${wheelWidth}" />
+                <xacro:property name="r" value="${diam/2}" />
+                <xacro:property name="h" value="${width}" />
                 <xacro:property name="m" value="${mass}" />
                 <mass value="${m}" />
@@ -126,6 +128,35 @@
         </gazebo>
     </xacro:macro>
-    <xacro:wheel prefix="front" suffix="left" origX="${wheelToMiddleLength}" origY="${wheelToMiddleWidth}" origZ="0.0" mass="${wheelWeight}"/>
-    <xacro:wheel prefix="front" suffix="right" origX="${wheelToMiddleLength}" origY="${-wheelToMiddleWidth}" origZ="0.0" mass="${wheelWeight}"/>
+    <xacro:wheel prefix="rear" suffix="left" origX="${-wheelToMiddleLength}" origY="${wheelToMiddleWidth}" origZ="0.0" mass="${wheelWeight}" diam="0.01" width="0.01"/>
+    <xacro:wheel prefix="rear" suffix="right" origX="${-wheelToMiddleLength}" origY="${-wheelToMiddleWidth}" origZ="0.0" mass="${wheelWeight}" diam="0.01" width="0.01"/>
+    <xacro:wheel prefix="front" suffix="left" origX="${wheelToMiddleLength}" origY="${wheelToMiddleWidth}" origZ="-0.02" mass="${wheelWeight}" diam="${wheelDiam}" width="${wheelWidth}"/>
+    <xacro:wheel prefix="front" suffix="right" origX="${wheelToMiddleLength}" origY="${-wheelToMiddleWidth}" origZ="-0.02" mass="${wheelWeight}" diam="${wheelDiam}" width="${wheelWidth}"/>
+    <link name="caster_wheel">
+        <visual>
+            <geometry>
+                <sphere radius="${casterWheelRadius}"/>
+            </geometry>
+            <material name="gray"/>
+        </visual>
+        <inertial>
+            <xacro:property name="r" value="${casterWheelRadius}" />
+            <xacro:property name="m" value="${casterWheelWeight}" />
+            <mass value="${m}" />
+            <inertia ixx="${(2/5)*m*r*r}" ixy="0.0" ixz="0.0"
+                     iyy="${(2/5)*m*r*r}" iyz="0.0"
+                     izz="${(2/5)*m*r*r}" />
+        </inertial>
+        <collision>
+            <geometry>
+                <sphere radius="${casterWheelRadius}"/>
+            </geometry>
+        </collision>
+    </link>
+    <joint name="base_caster_wheel_joint" type="fixed">
+        <axis rpy="0 0 0" xyz="0 1 0"/>
+        <parent link="base_link"/>
+        <child link="caster_wheel"/>
+        <origin rpy="0 0 0" xyz="-0.08 0 ${scale * -0.06}"/>
+    </joint>
     <gazebo>
         <plugin name="gazebo_ros_control" filename="libgazebo_ros_control.so">

Commit message: Add the second castor wheels, tweak the wheels' friction, decrease the
      ... spawn height

File: topnav_bot_description/urdf/capo2/capo2.urdf.xacro (robot description, xacro)
@@ -8,5 +8,5 @@
     <xacro:property name="caseWeight" value="${4 * scale}"/>
     <xacro:property name="wheelDiam" value="${0.1 * scale}" />
-    <xacro:property name="wheelWidth" value="${0.005 * scale}"/>
+    <xacro:property name="wheelWidth" value="${0.02 * scale}"/>
     <xacro:property name="wheelCaseGap" value="${0.0008 * scale}"/>
     <xacro:property name="wheelToMiddleWidth" value="${(caseWidth + wheelWidth)/2 + wheelCaseGap}"/>
@@ -15,5 +15,5 @@
     <xacro:property name="headDiam" value="${0.05 * scale}" />
     <xacro:property name="headHeight" value="${0.08 * scale}" />
-    <xacro:property name="headWeight" value="${0.2 * scale}" />
+    <xacro:property name="headWeight" value="${0.1 * scale}" />
     <xacro:property name="cameraWidth" value="${0.095 * scale}" />
     <xacro:property name="cameraHeight" value="${0.03 * scale}" />
@@ -22,5 +22,5 @@
     <xacro:property name="hokuyoHeight" value="${0.07 * scale}" />
     <xacro:property name="casterWheelRadius" value="${0.01 * scale}"/>
-    <xacro:property name="casterWheelWeight" value="${0.005 * scale}"/>
+    <xacro:property name="casterWheelWeight" value="${0.1* scale}"/>
     <xacro:property name="laserSamplesCount" value="61"/>
     <xacro:property name="laserMinAngle" value="${-2*pi/3}"/>
@@ -120,6 +120,6 @@
             <!-- generates warn  Element[mu], child of element[link] not defined in SDF. Ignoring[mu]-->
             <!-- http://wiki.ros.org/urdf/Tutorials/Using%20a%20URDF%20in%20Gazebo -->
-            <mu value="4.0"/>
-            <mu2 value="1.0"/>
+            <mu1 value="40.0"/>
+            <mu2 value="20.0"/>
             <kp value="1000000.0" />
             <kd value="1.0" />
@@ -132,31 +132,45 @@
     <xacro:wheel prefix="front" suffix="left" origX="${wheelToMiddleLength}" origY="${wheelToMiddleWidth}" origZ="-0.02" mass="${wheelWeight}" diam="${wheelDiam}" width="${wheelWidth}"/>
     <xacro:wheel prefix="front" suffix="right" origX="${wheelToMiddleLength}" origY="${-wheelToMiddleWidth}" origZ="-0.02" mass="${wheelWeight}" diam="${wheelDiam}" width="${wheelWidth}"/>
-    <link name="caster_wheel">
-        <visual>
-            <geometry>
-                <sphere radius="${casterWheelRadius}"/>
-            </geometry>
-            <material name="gray"/>
-        </visual>
-        <inertial>
-            <xacro:property name="r" value="${casterWheelRadius}" />
-            <xacro:property name="m" value="${casterWheelWeight}" />
-            <mass value="${m}" />
-            <inertia ixx="${(2/5)*m*r*r}" ixy="0.0" ixz="0.0"
-                     iyy="${(2/5)*m*r*r}" iyz="0.0"
-                     izz="${(2/5)*m*r*r}" />
-        </inertial>
-        <collision>
-            <geometry>
-                <sphere radius="${casterWheelRadius}"/>
-            </geometry>
-        </collision>
-    </link>
-    <joint name="base_caster_wheel_joint" type="fixed">
-        <axis rpy="0 0 0" xyz="0 1 0"/>
-        <parent link="base_link"/>
-        <child link="caster_wheel"/>
-        <origin rpy="0 0 0" xyz="-0.08 0 ${scale * -0.06}"/>
-    </joint>
+    <xacro:macro name="caster_wheel" params="prefix origX origY origZ">
+        <link name="${prefix}_caster_wheel">
+            <visual>
+                <geometry>
+                    <sphere radius="${casterWheelRadius}"/>
+                </geometry>
+                <material name="gray"/>
+            </visual>
+            <inertial>
+                <xacro:property name="r" value="${casterWheelRadius}"/>
+                <xacro:property name="m" value="${casterWheelWeight}"/>
+                <mass value="${m}"/>
+                <inertia ixx="${(2/5)*m*r*r}" ixy="0.0" ixz="0.0"
+                         iyy="${(2/5)*m*r*r}" iyz="0.0"
+                         izz="${(2/5)*m*r*r}"/>
+            </inertial>
+            <collision>
+                <geometry>
+                    <sphere radius="${casterWheelRadius}"/>
+                </geometry>
+                <surface>
+                    <friction>
+                        <ode>
+                            <mu>0</mu>
+                            <mu2>0</mu2>
+                            <slip1>1.0</slip1>
+                            <slip2>1.0</slip2>
+                        </ode>
+                    </friction>
+                </surface>
+            </collision>
+        </link>
+        <joint name="base_${prefix}_caster_wheel_joint" type="fixed">
+            <axis rpy="0 0 0" xyz="0 1 0"/>
+            <parent link="base_link"/>
+            <child link="${prefix}_caster_wheel"/>
+            <origin rpy="0 0 0" xyz="${origX} ${origY} ${origZ}"/>
+        </joint>
+    </xacro:macro>
+    <xacro:caster_wheel prefix="left" origX="-0.08" origY="0.04" origZ="${scale * -0.06}"/>
+    <xacro:caster_wheel prefix="right" origX="-0.08" origY="-0.04" origZ="${scale * -0.06}"/>
     <gazebo>
         <plugin name="gazebo_ros_control" filename="libgazebo_ros_control.so">

Commit message: Replace the HS-422 servo, change the upper servo's target range
      * Add the scaffold fot the Pololu wheels (TODO sdf model)

File: topnav_bot_description/urdf/capo2/capo2.urdf.xacro (robot description, xacro)
@@ -129,4 +129,5 @@
             <!--<fdir1>0 0 1</fdir1>-->
             <material>Gazebo/Black</material>
+            <!--<material>Topnav/PololuWheel</material>-->
         </gazebo>
     </xacro:macro>

Commit message: Add another test, tweak the capo2 model
      * Compensate the battery weight by increasing the castor wheel
      weight
      * Change the texture of the wheel for the debugging purposes

File: topnav_bot_description/urdf/capo2/capo2.urdf.xacro (robot description, xacro)
@@ -26,5 +26,5 @@
     <xacro:property name="hokuyoHeightOffset" value="${0.03 * scale}" />
     <xacro:property name="casterWheelRadius" value="${0.01 * scale}"/>
-    <xacro:property name="casterWheelWeight" value="${0.1* scale}"/>
+    <xacro:property name="casterWheelWeight" value="${1.0 * scale}"/>
     <xacro:property name="laserSamplesCount" value="61"/>
     <xacro:property name="laserMinAngle" value="${-2*pi/3}"/>
@@ -135,5 +135,6 @@
             <kd value="1.0" />
             <!--<fdir1>0 0 1</fdir1>-->
-            <material>Gazebo/Black</material>
+            <!--<material>Gazebo/Black</material>-->
+            <material>Gazebo/Wood</material>
             <!--<material>Topnav/PololuWheel</material>-->
         </gazebo>

Commit message: Change the simulated camera FOV, do not visualize the laser beams

File: topnav_bot_description/urdf/capo2/capo2.urdf.xacro (robot description, xacro)
@@ -30,4 +30,5 @@
     <xacro:property name="laserMinAngle" value="${-2*pi/3}"/>
     <xacro:property name="laserMaxAngle" value="${2*pi/3}"/>
+    <xacro:property name="visualizeLaser" value="false" />
     <xacro:if value="$(arg use_real_camera)">
         <xacro:property name="cameraFileName" value="camera_real.gazebo" />

Commit message: Improve the inertial parameters, fix robot's skidding on moving back
      * Remove the mass from the inertia matrix
      * Place the rear wheels in the same axis as the front wheels

File: topnav_bot_description/urdf/capo2/capo2.urdf.xacro (robot description, xacro)
@@ -20,4 +20,5 @@
     <xacro:property name="wheelToMiddleLength" value="${caseLength/2 - 0.06 * scale}"/>
     <xacro:property name="wheelWeight" value="${0.15 * scale}" />
+    <xacro:property name="smallWheelWeight" value="${0.001 * scale}" />
     <xacro:property name="headDiam" value="${0.05 * scale}" />
     <xacro:property name="headHeight" value="${0.08 * scale}" />
@@ -32,5 +33,5 @@
     <xacro:property name="hokuyoHeightOffset" value="${0.03 * scale}" />
     <xacro:property name="casterWheelRadius" value="${0.01 * scale}"/>
-    <xacro:property name="casterWheelWeight" value="${0.5 * scale}"/>
+    <xacro:property name="casterWheelWeight" value="${0.05 * scale}"/>
     <xacro:property name="laserSamplesCount" value="61"/>
     <xacro:property name="laserMinAngle" value="${-2*pi/3}"/>
@@ -59,12 +60,12 @@
         </visual>
         <inertial>
+            <xacro:property name="d" value="${caseLength}" />
             <xacro:property name="w" value="${caseWidth}" />
             <xacro:property name="h" value="${caseHeight}" />
-            <xacro:property name="d" value="${caseLength}" />
             <xacro:property name="m" value="${caseWeight}" />
             <mass value="${m}" />
-            <inertia ixx="${(1/12)*m*(h*h+d*d)}" ixy="0.0" ixz="0.0"
-                     iyy="${(1/12)*m*(w*w+h*h)}" iyz="0.0"
-                     izz="${(1/12)*m*(w*w+d*d)}" />
+            <inertia ixx="${(1/12)*(h*h+w*w)}" ixy="0.0" ixz="0.0"
+                     iyy="${(1/12)*(d*d+h*h)}" iyz="0.0"
+                     izz="${(1/12)*(w*w+d*d)}" />
         </inertial>
         <collision>
@@ -86,12 +87,12 @@
         </visual>
         <inertial>
+            <xacro:property name="d" value="${batteryLength}" />
             <xacro:property name="w" value="${batteryWidth}" />
             <xacro:property name="h" value="${batteryHeight}" />
-            <xacro:property name="d" value="${batteryLength}" />
             <xacro:property name="m" value="${batteryWeight}" />
             <mass value="${m}" />
-            <inertia ixx="${(1/12)*m*(h*h+d*d)}" ixy="0.0" ixz="0.0"
-                     iyy="${(1/12)*m*(w*w+h*h)}" iyz="0.0"
-                     izz="${(1/12)*m*(w*w+d*d)}" />
+           <inertia ixx="${(1/12)*(h*h+w*w)}" ixy="0.0" ixz="0.0"
+                     iyy="${(1/12)*(d*d+h*h)}" iyz="0.0"
+                     izz="${(1/12)*(w*w+d*d)}" />
         </inertial>
         <collision>
@@ -151,7 +152,7 @@
                 <xacro:property name="m" value="${mass}" />
                 <mass value="${m}" />
-                <inertia ixx="${(1/12)*m*(3*r*r+h*h)}" ixy="0.0" ixz="0.0"
-                         iyy="${0.5*m*r*r}" iyz="0.0"
-                         izz="${(1/12)*m*(3*r*r+h*h)}" />
+                <inertia ixx="${(1/12)*(3*r*r+h*h)}" ixy="0.0" ixz="0.0"
+                         iyy="${(1/2)*r*r}" iyz="0.0"
+                         izz="${(1/12)*(3*r*r+h*h)}"/>
             </inertial>
         </link>
@@ -184,6 +185,6 @@
         </gazebo>
     </xacro:macro>
-    <xacro:wheel prefix="rear" suffix="left" origX="${-wheelToMiddleLength}" origY="${wheelToMiddleWidth}" origZ="0.0" mass="${wheelWeight * 0.0001}" diam="0.01" width="0.01"/>
-    <xacro:wheel prefix="rear" suffix="right" origX="${-wheelToMiddleLength}" origY="${-wheelToMiddleWidth}" origZ="0.0" mass="${wheelWeight * 0.0001}" diam="0.01" width="0.01"/>
+    <xacro:wheel prefix="rear" suffix="left" origX="${wheelToMiddleLength}" origY="${wheelToMiddleWidth + wheelWidth}" origZ="-0.025" mass="${smallWheelWeight}" diam="0.01" width="0.005"/>
+    <xacro:wheel prefix="rear" suffix="right" origX="${wheelToMiddleLength}" origY="${-wheelToMiddleWidth - wheelWidth}" origZ="-0.025" mass="${smallWheelWeight}" diam="0.01" width="0.005"/>
     <xacro:wheel prefix="front" suffix="left" origX="${wheelToMiddleLength}" origY="${wheelToMiddleWidth}" origZ="-0.025" mass="${wheelWeight}" diam="${wheelDiam}" width="${wheelWidth}"/>
     <xacro:wheel prefix="front" suffix="right" origX="${wheelToMiddleLength}" origY="${-wheelToMiddleWidth}" origZ="-0.025" mass="${wheelWeight}" diam="${wheelDiam}" width="${wheelWidth}"/>
@@ -200,7 +201,7 @@
                 <xacro:property name="m" value="${casterWheelWeight}"/>
                 <mass value="${m}"/>
-                <inertia ixx="${(2/5)*m*r*r}" ixy="0.0" ixz="0.0"
-                         iyy="${(2/5)*m*r*r}" iyz="0.0"
-                         izz="${(2/5)*m*r*r}"/>
+                <inertia ixx="${(2/5)*r*r}" ixy="0.0" ixz="0.0"
+                         iyy="${(2/5)*r*r}" iyz="0.0"
+                         izz="${(2/5)*r*r}"/>
             </inertial>
             <collision>
