Commit message: Fix/fricion skidding inertia (#21)
* Change the simulated camera FOV, do not visualize the laser beams

* Add the battery, tweak the masses and the inertial values

* Improve the inertial parameters, fix robot's skidding on moving back

      * Remove the mass from the inertia matrix
      * Place the rear wheels in the same axis as the front wheels

* Apply the review changes

File: topnav_bot_description/urdf/capo2/capo2.urdf.xacro (robot description, xacro)
@@ -7,5 +7,11 @@
     <xacro:property name="caseLength" value="${0.18 * scale}" />
     <xacro:property name="caseHeight" value="${0.12 * scale}" />
-    <xacro:property name="caseWeight" value="${4 * scale}"/>
+    <xacro:property name="caseWeight" value="${1.0 * scale}"/>
+    <xacro:property name="batteryWidth" value="${0.13 * scale}" />
+    <xacro:property name="batteryLength" value="${0.04 * scale}" />
+    <xacro:property name="batteryHeight" value="${0.05 * scale}" />
+    <xacro:property name="batteryWeight" value="${0.5 * scale}"/>
+    <xacro:property name="batteryOffset" value="${-0.065 * scale}" />
+    <xacro:property name="batteryHeightOffset" value="${-0.03 * scale}" />
     <xacro:property name="wheelDiam" value="${0.09 * scale}" />
     <xacro:property name="wheelWidth" value="${0.01 * scale}"/>
@@ -14,4 +20,5 @@
     <xacro:property name="wheelToMiddleLength" value="${caseLength/2 - 0.06 * scale}"/>
     <xacro:property name="wheelWeight" value="${0.15 * scale}" />
+    <xacro:property name="smallWheelWeight" value="${0.001 * scale}" />
     <xacro:property name="headDiam" value="${0.05 * scale}" />
     <xacro:property name="headHeight" value="${0.08 * scale}" />
@@ -26,8 +33,9 @@
     <xacro:property name="hokuyoHeightOffset" value="${0.03 * scale}" />
     <xacro:property name="casterWheelRadius" value="${0.01 * scale}"/>
-    <xacro:property name="casterWheelWeight" value="${1.0 * scale}"/>
+    <xacro:property name="casterWheelWeight" value="${0.05 * scale}"/>
     <xacro:property name="laserSamplesCount" value="61"/>
     <xacro:property name="laserMinAngle" value="${-2*pi/3}"/>
     <xacro:property name="laserMaxAngle" value="${2*pi/3}"/>
+    <xacro:property name="visualizeLaser" value="false" />
     <xacro:if value="$(arg use_real_camera)">
         <xacro:property name="cameraFileName" value="camera_real.gazebo" />
@@ -52,12 +60,12 @@
         </visual>
         <inertial>
+            <xacro:property name="d" value="${caseLength}" />
             <xacro:property name="w" value="${caseWidth}" />
             <xacro:property name="h" value="${caseHeight}" />
-            <xacro:property name="d" value="${caseLength}" />
             <xacro:property name="m" value="${caseWeight}" />
             <mass value="${m}" />
-            <inertia ixx="${(1/12)*m*(h*h+d*d)}" ixy="0.0" ixz="0.0"
-                     iyy="${(1/12)*m*(w*w+h*h)}" iyz="0.0"
-                     izz="${(1/12)*m*(w*w+d*d)}" />
+            <inertia ixx="${(1/12)*(h*h+w*w)}" ixy="0.0" ixz="0.0"
+                     iyy="${(1/12)*(d*d+h*h)}" iyz="0.0"
+                     izz="${(1/12)*(w*w+d*d)}" />
         </inertial>
         <collision>
@@ -67,4 +75,41 @@
         </collision>
     </link>
+    <gazebo reference="base_link">
+        <material>Gazebo/Wood</material>
+    </gazebo>
+    <!--battery -->
+    <link name ="battery">
+        <visual>
+            <geometry>
+                <box size="${batteryLength} ${batteryWidth} ${batteryHeight}"/>
+            </geometry>
+            <material name="gray"/>
+        </visual>
+        <inertial>
+            <xacro:property name="d" value="${batteryLength}" />
+            <xacro:property name="w" value="${batteryWidth}" />
+            <xacro:property name="h" value="${batteryHeight}" />
+            <xacro:property name="m" value="${batteryWeight}" />
+            <mass value="${m}" />
+           <inertia ixx="${(1/12)*(h*h+w*w)}" ixy="0.0" ixz="0.0"
+                     iyy="${(1/12)*(d*d+h*h)}" iyz="0.0"
+                     izz="${(1/12)*(w*w+d*d)}" />
+        </inertial>
+        <collision>
+            <geometry>
+                <box size="${batteryLength} ${batteryWidth} ${batteryHeight}"/>
+            </geometry>
+        </collision>
+    </link>
+    <joint name="base_battery_joint" type="fixed">
+        <axis rpy="0 0 0" xyz="0 1 0"/>
+        <parent link="base_link"/>
+        <child link="battery"/>
+        <origin rpy="0 0 0" xyz="${batteryOffset} 0.0 ${batteryHeightOffset}"/>
+    </joint>
+    <gazebo reference="battery">
+        <material>Gazebo/Blue</material>
+    </gazebo>
+    <!-- battery -->
     <xacro:include filename="../capo/head/capo.head.xacro" />
     <transmission name="head_swivel_trans">
@@ -107,7 +152,7 @@
                 <xacro:property name="m" value="${mass}" />
                 <mass value="${m}" />
-                <inertia ixx="${(1/12)*m*(3*r*r+h*h)}" ixy="0.0" ixz="0.0"
-                         iyy="${0.5*m*r*r}" iyz="0.0"
-                         izz="${(1/12)*m*(3*r*r+h*h)}" />
+                <inertia ixx="${(1/12)*(3*r*r+h*h)}" ixy="0.0" ixz="0.0"
+                         iyy="${(1/2)*r*r}" iyz="0.0"
+                         izz="${(1/12)*(3*r*r+h*h)}"/>
             </inertial>
         </link>
@@ -132,5 +177,5 @@
             <mu1 value="40.0"/>
             <mu2 value="20.0"/>
-            <kp value="1000000.0" />
+            <kp value="10000000.0" />
             <kd value="1.0" />
             <!--<fdir1>0 0 1</fdir1>-->
@@ -140,6 +185,6 @@
         </gazebo>
     </xacro:macro>
-    <xacro:wheel prefix="rear" suffix="left" origX="${-wheelToMiddleLength}" origY="${wheelToMiddleWidth}" origZ="0.0" mass="${wheelWeight}" diam="0.01" width="0.01"/>
-    <xacro:wheel prefix="rear" suffix="right" origX="${-wheelToMiddleLength}" origY="${-wheelToMiddleWidth}" origZ="0.0" mass="${wheelWeight}" diam="0.01" width="0.01"/>
+    <xacro:wheel prefix="rear" suffix="left" origX="${wheelToMiddleLength}" origY="${wheelToMiddleWidth + wheelWidth}" origZ="-0.025" mass="${smallWheelWeight}" diam="0.01" width="0.005"/>
+    <xacro:wheel prefix="rear" suffix="right" origX="${wheelToMiddleLength}" origY="${-wheelToMiddleWidth - wheelWidth}" origZ="-0.025" mass="${smallWheelWeight}" diam="0.01" width="0.005"/>
     <xacro:wheel prefix="front" suffix="left" origX="${wheelToMiddleLength}" origY="${wheelToMiddleWidth}" origZ="-0.025" mass="${wheelWeight}" diam="${wheelDiam}" width="${wheelWidth}"/>
     <xacro:wheel prefix="front" suffix="right" origX="${wheelToMiddleLength}" origY="${-wheelToMiddleWidth}" origZ="-0.025" mass="${wheelWeight}" diam="${wheelDiam}" width="${wheelWidth}"/>
@@ -156,7 +201,7 @@
                 <xacro:property name="m" value="${casterWheelWeight}"/>
                 <mass value="${m}"/>
-                <inertia ixx="${(2/5)*m*r*r}" ixy="0.0" ixz="0.0"
-                         iyy="${(2/5)*m*r*r}" iyz="0.0"
-                         izz="${(2/5)*m*r*r}"/>
+                <inertia ixx="${(2/5)*r*r}" ixy="0.0" ixz="0.0"
+                         iyy="${(2/5)*r*r}" iyz="0.0"
+                         izz="${(2/5)*r*r}"/>
             </inertial>
             <collision>
@@ -183,6 +228,5 @@
         </joint>
     </xacro:macro>
-    <xacro:caster_wheel prefix="left" origX="-0.08" origY="0.04" origZ="${scale * -0.06}"/>
-    <xacro:caster_wheel prefix="right" origX="-0.08" origY="-0.04" origZ="${scale * -0.06}"/>
+    <xacro:caster_wheel prefix="center" origX="-0.08" origY="0.0" origZ="${scale * -0.06}"/>
     <gazebo>
         <plugin name="gazebo_ros_control" filename="libgazebo_ros_control.so">

Commit message: Feature/marker trackin with latency (#19)
* Increase the servo speed

* Set the wheels acceleration

* Fix - method name

* Add the launch file

* Remove the timeout

* Set the initial head rotation to 0.0

* Add another test, tweak the capo2 model

      * Compensate the battery weight by increasing the castor wheel
      weight
      * Change the texture of the wheel for the debugging purposes

* Add the debug print

* Surround the head rotation reading with try except

* Comment out the acceleration setting and setting the target to 0

* Tweak the wheels target ranges

* Specify the speed and acceleration

* Download maestro

* Add the test_maestro

* Change the channel of the wheel servo

* Switch back to 0 and 1 for the wheel servos

* Revert 0 target setting

* Handle error

* Add head servo test

* Test head and wheels

* Separate read from write

* Re-raise the exception

* Delay the node start

* Move the wheel-servo speed and acceleration to the constants

* Decrease the velocity coefficient

* Filter out the noise

* Increase the coefficient

* Decrease the coefficient

* Add the capo2's clock publisher

* Allow to parametrize the clock publish rate via launch file

* Change to the unsigned int64

* Run the capo2 clock in the gazebo simulations

* Change the simulated camera FOV, do not visualize the laser beams

* Fix/fricion skidding inertia (#21)

* Change the simulated camera FOV, do not visualize the laser beams

* Add the battery, tweak the masses and the inertial values

* Improve the inertial parameters, fix robot's skidding on moving back

      * Remove the mass from the inertia matrix
      * Place the rear wheels in the same axis as the front wheels

* Apply the review changes

* Print info about shutting down the clock instead of the stacktrace

File: topnav_bot_description/urdf/capo2/capo2.urdf.xacro (robot description, xacro)
@@ -7,5 +7,11 @@
     <xacro:property name="caseLength" value="${0.18 * scale}" />
     <xacro:property name="caseHeight" value="${0.12 * scale}" />
-    <xacro:property name="caseWeight" value="${4 * scale}"/>
+    <xacro:property name="caseWeight" value="${1.0 * scale}"/>
+    <xacro:property name="batteryWidth" value="${0.13 * scale}" />
+    <xacro:property name="batteryLength" value="${0.04 * scale}" />
+    <xacro:property name="batteryHeight" value="${0.05 * scale}" />
+    <xacro:property name="batteryWeight" value="${0.5 * scale}"/>
+    <xacro:property name="batteryOffset" value="${-0.065 * scale}" />
+    <xacro:property name="batteryHeightOffset" value="${-0.03 * scale}" />
     <xacro:property name="wheelDiam" value="${0.09 * scale}" />
     <xacro:property name="wheelWidth" value="${0.01 * scale}"/>
@@ -14,4 +20,5 @@
     <xacro:property name="wheelToMiddleLength" value="${caseLength/2 - 0.06 * scale}"/>
     <xacro:property name="wheelWeight" value="${0.15 * scale}" />
+    <xacro:property name="smallWheelWeight" value="${0.001 * scale}" />
     <xacro:property name="headDiam" value="${0.05 * scale}" />
     <xacro:property name="headHeight" value="${0.08 * scale}" />
@@ -26,8 +33,9 @@
     <xacro:property name="hokuyoHeightOffset" value="${0.03 * scale}" />
     <xacro:property name="casterWheelRadius" value="${0.01 * scale}"/>
-    <xacro:property name="casterWheelWeight" value="${0.1* scale}"/>
+    <xacro:property name="casterWheelWeight" value="${0.05 * scale}"/>
     <xacro:property name="laserSamplesCount" value="61"/>
     <xacro:property name="laserMinAngle" value="${-2*pi/3}"/>
     <xacro:property name="laserMaxAngle" value="${2*pi/3}"/>
+    <xacro:property name="visualizeLaser" value="false" />
     <xacro:if value="$(arg use_real_camera)">
         <xacro:property name="cameraFileName" value="camera_real.gazebo" />
@@ -52,12 +60,12 @@
         </visual>
         <inertial>
+            <xacro:property name="d" value="${caseLength}" />
             <xacro:property name="w" value="${caseWidth}" />
             <xacro:property name="h" value="${caseHeight}" />
-            <xacro:property name="d" value="${caseLength}" />
             <xacro:property name="m" value="${caseWeight}" />
             <mass value="${m}" />
-            <inertia ixx="${(1/12)*m*(h*h+d*d)}" ixy="0.0" ixz="0.0"
-                     iyy="${(1/12)*m*(w*w+h*h)}" iyz="0.0"
-                     izz="${(1/12)*m*(w*w+d*d)}" />
+            <inertia ixx="${(1/12)*(h*h+w*w)}" ixy="0.0" ixz="0.0"
+                     iyy="${(1/12)*(d*d+h*h)}" iyz="0.0"
+                     izz="${(1/12)*(w*w+d*d)}" />
         </inertial>
         <collision>
@@ -67,4 +75,41 @@
         </collision>
     </link>
+    <gazebo reference="base_link">
+        <material>Gazebo/Wood</material>
+    </gazebo>
+    <!--battery -->
+    <link name ="battery">
+        <visual>
+            <geometry>
+                <box size="${batteryLength} ${batteryWidth} ${batteryHeight}"/>
+            </geometry>
+            <material name="gray"/>
+        </visual>
+        <inertial>
+            <xacro:property name="d" value="${batteryLength}" />
+            <xacro:property name="w" value="${batteryWidth}" />
+            <xacro:property name="h" value="${batteryHeight}" />
+            <xacro:property name="m" value="${batteryWeight}" />
+            <mass value="${m}" />
+           <inertia ixx="${(1/12)*(h*h+w*w)}" ixy="0.0" ixz="0.0"
+                     iyy="${(1/12)*(d*d+h*h)}" iyz="0.0"
+                     izz="${(1/12)*(w*w+d*d)}" />
+        </inertial>
+        <collision>
+            <geometry>
+                <box size="${batteryLength} ${batteryWidth} ${batteryHeight}"/>
+            </geometry>
+        </collision>
+    </link>
+    <joint name="base_battery_joint" type="fixed">
+        <axis rpy="0 0 0" xyz="0 1 0"/>
+        <parent link="base_link"/>
+        <child link="battery"/>
+        <origin rpy="0 0 0" xyz="${batteryOffset} 0.0 ${batteryHeightOffset}"/>
+    </joint>
+    <gazebo reference="battery">
+        <material>Gazebo/Blue</material>
+    </gazebo>
+    <!-- battery -->
     <xacro:include filename="../capo/head/capo.head.xacro" />
     <transmission name="head_swivel_trans">
@@ -107,7 +152,7 @@
                 <xacro:property name="m" value="${mass}" />
                 <mass value="${m}" />
-                <inertia ixx="${(1/12)*m*(3*r*r+h*h)}" ixy="0.0" ixz="0.0"
-                         iyy="${0.5*m*r*r}" iyz="0.0"
-                         izz="${(1/12)*m*(3*r*r+h*h)}" />
+                <inertia ixx="${(1/12)*(3*r*r+h*h)}" ixy="0.0" ixz="0.0"
+                         iyy="${(1/2)*r*r}" iyz="0.0"
+                         izz="${(1/12)*(3*r*r+h*h)}"/>
             </inertial>
         </link>
@@ -132,13 +177,14 @@
             <mu1 value="40.0"/>
             <mu2 value="20.0"/>
-            <kp value="1000000.0" />
+            <kp value="10000000.0" />
             <kd value="1.0" />
             <!--<fdir1>0 0 1</fdir1>-->
-            <material>Gazebo/Black</material>
+            <!--<material>Gazebo/Black</material>-->
+            <material>Gazebo/Wood</material>
             <!--<material>Topnav/PololuWheel</material>-->
         </gazebo>
     </xacro:macro>
-    <xacro:wheel prefix="rear" suffix="left" origX="${-wheelToMiddleLength}" origY="${wheelToMiddleWidth}" origZ="0.0" mass="${wheelWeight}" diam="0.01" width="0.01"/>
-    <xacro:wheel prefix="rear" suffix="right" origX="${-wheelToMiddleLength}" origY="${-wheelToMiddleWidth}" origZ="0.0" mass="${wheelWeight}" diam="0.01" width="0.01"/>
+    <xacro:wheel prefix="rear" suffix="left" origX="${wheelToMiddleLength}" origY="${wheelToMiddleWidth + wheelWidth}" origZ="-0.025" mass="${smallWheelWeight}" diam="0.01" width="0.005"/>
+    <xacro:wheel prefix="rear" suffix="right" origX="${wheelToMiddleLength}" origY="${-wheelToMiddleWidth - wheelWidth}" origZ="-0.025" mass="${smallWheelWeight}" diam="0.01" width="0.005"/>
     <xacro:wheel prefix="front" suffix="left" origX="${wheelToMiddleLength}" origY="${wheelToMiddleWidth}" origZ="-0.025" mass="${wheelWeight}" diam="${wheelDiam}" width="${wheelWidth}"/>
     <xacro:wheel prefix="front" suffix="right" origX="${wheelToMiddleLength}" origY="${-wheelToMiddleWidth}" origZ="-0.025" mass="${wheelWeight}" diam="${wheelDiam}" width="${wheelWidth}"/>
@@ -155,7 +201,7 @@
                 <xacro:property name="m" value="${casterWheelWeight}"/>
                 <mass value="${m}"/>
-                <inertia ixx="${(2/5)*m*r*r}" ixy="0.0" ixz="0.0"
-                         iyy="${(2/5)*m*r*r}" iyz="0.0"
-                         izz="${(2/5)*m*r*r}"/>
+                <inertia ixx="${(2/5)*r*r}" ixy="0.0" ixz="0.0"
+                         iyy="${(2/5)*r*r}" iyz="0.0"
+                         izz="${(2/5)*r*r}"/>
             </inertial>
             <collision>
@@ -182,6 +228,5 @@
         </joint>
     </xacro:macro>
-    <xacro:caster_wheel prefix="left" origX="-0.08" origY="0.04" origZ="${scale * -0.06}"/>
-    <xacro:caster_wheel prefix="right" origX="-0.08" origY="-0.04" origZ="${scale * -0.06}"/>
+    <xacro:caster_wheel prefix="center" origX="-0.08" origY="0.0" origZ="${scale * -0.06}"/>
     <gazebo>
         <plugin name="gazebo_ros_control" filename="libgazebo_ros_control.so">
